File: kicad/esp8266.kicad_pcb (KiCad board)
At the start: 2 copper layers, 85 x 75 mm, 62 parts, among them J1 BATT, J10 Green, J11 Blue, J12 White, J13 IO_RGBW, J14 +12V, J15 hole, J16 hole, J17 hole, J18 hole, J2 5 / 12V, J3 CONN FT232RL, J4 RJ12-I2C, J5 RJ12-I2C, J6 Onewire, J7 Onewire, J8 Red, J9 Pad, Q1 BSP75, Q2 BSP75, Q3 BSP75, Q4 BSP75, SW1 RESET, SW2 PROG, U1 ESP-12E, U2 MCP73831-2, U3 MCP1703-33, U4 MS5637, U5 MCP1703-50, U6 Si7020-A20, U7 DS18B20

Commit message: work in progress
Parts:
- U1: value ESP-12E -> ESP32-WROOM-32U; footprint RF_Module:ESP-12E -> RF_Module:ESP32-WROOM-32U
- moved R11 11.4 mm to (133.9, 101.4)
- moved U1 5.32 mm to (128.8, 79.8)
Connections:
- SW2 pad 1: Net-(R10-Pad2) -> GND
- SW2 pad 2: GND -> Net-(R10-Pad2)
- U1 pad 1: /RST -> GND
- U1 pad 12: Net-(U1-Pad12) -> /ADC
- U1 pad 13: Net-(U1-Pad13) -> /IO14
- U1 pad 14: Net-(U1-Pad14) -> /IO12
- U1 pad 16: /IO15 -> /IO13
- U1 pad 17: /IO2 -> Net-(U1-Pad17)
- U1 pad 18: Net-(R10-Pad2) -> Net-(U1-Pad18)
- U1 pad 19: /SDA -> Net-(U1-Pad19)
- U1 pad 2: /ADC -> +3V3
- U1 pad 20: /SCL -> Net-(U1-Pad20)
- U1 pad 21: /RX -> Net-(R10-Pad2)
- U1 pad 22: /TX -> Net-(U1-Pad22)
- U1 pad 3: /EN -> /RST
- U1 pad 4: /RST -> Net-(U1-Pad4)
- U1 pad 5: /IO14 -> Net-(U1-Pad5)
- U1 pad 6: /IO12 -> /ONE1
- U1 pad 7: /IO13 -> /ONE2
- U1 pad 8: +3V3 -> Net-(U1-Pad8)
Routing:
- net /RST: track 54.8 -> 17.8 mm
- net /IO13: track 57.9 -> 22.2 mm
- net /IO14: track 50.1 -> 16.4 mm
- net +3V3: track 160.7 -> 130.7 mm
- net /IO12: track 54.7 -> 29.4 mm
- net Net-(R10-Pad2): track 39.7 -> 14.9 mm
- net /SDA: track 238.7 -> 215.0 mm
- net /RX: track 60.4 -> 38.8 mm, vias 2 -> 1
- net /IO15: track 46.8 -> 26.7 mm
- net /TX: track 62.5 -> 43.2 mm, vias 1 -> 0
- net /SCL: track 255.6 -> 248.5 mm
- net GND: track 115.8 -> 109.0 mm, vias 14 -> 13
- net /ADC: track 11.2 -> 5.08 mm
- net /EN: track 5.11 -> 0.00 mm
- net /IO2: track 77.2 -> 73.7 mm
Other:
- board size 85 x 75 mm -> 85.1 x 75 mm
