File: kicad/esp8266.sch (KiCad schematic (older format))
At the start: 43 parts, among them J10 Green, J11 Blue, J12 White, J13 IO_RGBW, J14 +12V, J15 hole, J16 hole, J17 hole, J18 hole, J2 5 / 12V, J3 CONN FT232RL, J4 RJ12-I2C, J5 RJ12-I2C, J6 Onewire, J7 Onewire, J8 Red, J9 Pad, Q1 BSP75, Q2 BSP75, Q3 BSP75, Q4 BSP75, SW1 RESET, SW2 PROG, U1 ESP-12E, U4 MS5637, U6 Si7020-A20, U7 DS18B20

Commit message: work in progress
Parts:
- removed R10, R11, R7, R8: 10k, Resistor_SMD:R_0805_2012Metric_Pad1.15x1.40mm_HandSolder, symbol Device:R
- removed U1: ESP-12E, RF_Module:ESP-12E, symbol RF_Module:ESP-12E
- added C10, C?: 100nF, symbol Device:C
- added R?: 499, symbol Device:R
- added U1: ESP32-WROOM-32U, RF_Module:ESP32-WROOM-32U, symbol RF_Module:ESP32-WROOM-32U
Connections:
- net labels added: IO34, IO35, ONE1, ONE2
- net labels removed: EN
- wire segments 116 -> 119
- no-connect marks 17 -> 12
Other:
- note removed: "Onewire\n"
- note removed: "USED BY FLASH"
