File: kicad/MCP73831.sch (KiCad schematic (older format))
At the start: 13 parts, among them J1 BATT, U2 MCP73831-2

Commit message: work in progress
Parts:
- D1: symbol esp8266-rescue:DMP1045U-DMP1045U -> esp32-rescue:DMP1045U-DMP1045U
Changed lines of the file:
@@
 EESchema Schematic File Version 4
-LIBS:esp8266-cache
+LIBS:esp32-cache
 EELAYER 26 0
 EELAYER END
@@
 	7100 3000 7100 3150
 $Comp
-L esp8266-rescue:DMP1045U-DMP1045U D1
+L esp32-rescue:DMP1045U-DMP1045U D1
 U 1 1 5C39EFFF
 P 8050 2700
