File: kicad/esp32.kicad_pcb (KiCad board)
At the start: 2 copper layers, 85.1 x 75 mm, 62 parts, among them J1 BATT, J10 Green, J11 Blue, J12 White, J13 IO_RGBW, J14 +12V, J15 hole, J16 hole, J17 hole, J18 hole, J2 5 / 12V, J3 CONN FT232RL, J4 RJ12-I2C, J5 RJ12-I2C, J6 Onewire, J7 Onewire, J8 Red, J9 Pad, Q1 BSP75, Q2 BSP75, Q3 BSP75, Q4 BSP75, SW1 RESET, SW2 PROG, U1 ESP32-WROOM-32U, U2 MCP73831-2, U3 MCP1703-33, U4 MS5637, U5 MCP1703-50, U6 Si7020-A20, U7 DS18B20

Commit message: work in progress
Parts:
- added C10: 100nF, Capacitor_SMD:C_0805_2012Metric_Pad1.15x1.40mm_HandSolder, F.Cu at (156.7, 69.1)
- added C11: 100nF, Capacitor_SMD:C_0805_2012Metric_Pad1.15x1.40mm_HandSolder, F.Cu at (156.7, 73.5)
- added D2: LED, LED_SMD:LED_0805_2012Metric_Pad1.15x1.40mm_HandSolder, F.Cu at (118.9, 102.7)
- added D5: LED, LED_SMD:LED_0805_2012Metric_Pad1.15x1.40mm_HandSolder, F.Cu at (141.3, 87.5)
- added R10: 10k, Resistor_SMD:R_0805_2012Metric_Pad1.15x1.40mm_HandSolder, F.Cu at (141.5, 90.0)
- added R7: 499, Resistor_SMD:R_0805_2012Metric_Pad1.15x1.40mm_HandSolder, F.Cu at (113.8, 64.6)
- added R8: 10k, Resistor_SMD:R_0805_2012Metric_Pad1.15x1.40mm_HandSolder, F.Cu at (119.0, 99.5)
Connections:
- J6 pad T: /IO2 -> /IO35
- J7 pad T: /IO2 -> /IO34
- SW2 pad 1: GND -> /IO0
- SW2 pad 2: Net-(R10-Pad2) -> GND
- U1 pad 21: Net-(R10-Pad2) -> Net-(U1-Pad21)
- U1 pad 25: Net-(U1-Pad25) -> /IO0
- U1 pad 35: /TX -> Net-(R7-Pad2)
Routing:
- net /RST: track 17.8 -> 45.2 mm
- net /SDA: track 215.0 -> 237.1 mm
- net /IO15: track 26.7 -> 13.1 mm
- net /SCL: track 248.5 -> 254.1 mm
- net /IO0: track 0.00 -> 5.25 mm
- net GND: track 109.0 -> 113.1 mm
Other:
- board size 85.1 x 75 mm -> 85 x 75 mm
- board text added: "ESP-32 Playground 1.0"
- board text removed: "ESP-12e Playground 1.0"

Commit message: chore: working on pcb
Parts:
- removed U7: DS18B20, Package_TO_SOT_THT:TO-92_Inline
- added R11: 4.7k, Resistor_SMD:R_0805_2012Metric_Pad1.15x1.40mm_HandSolder, F.Cu at (141.8, 111.3)
- added TP8: OneWire, TestPoint:TestPoint_2Pads_Pitch2.54mm_Drill0.8mm, F.Cu at (138.4, 107.2)
- C10: value 100nF -> 10uF
- moved C11 12.2 mm to (148.4, 82.4), turned to 0 degrees
- moved D5 5.09 mm to (141.5, 82.4)
- moved R10 5.08 mm to (141.5, 84.9)
- moved R7 0.52 mm to (114.3, 64.6)
- moved SW2 0.11 mm to (149.1, 76.8), turned to 180 degrees
Connections:
- J13 pad 4: /IO12 -> /EXT1
- J13 pad 5: /IO13 -> /EXT2
- J13 pad 6: /IO14 -> /EXT3
- J13 pad 7: /IO15 -> /EXT4
- J6 pad T: /IO35 -> /ONE2
- J7 pad T: /IO34 -> /ONE1
- R3 pad 2: /MCP73831/V_STATUS -> /CHARGING
- R4 pad 1: /MCP73831/V_STATUS -> /CHARGING
- R9 pad 2: /IO2 -> /ONE1
- TP3 pad 1: /IO2 -> /ONE1
- U1 pad 10: Net-(U1-Pad10) -> /EXT1
- U1 pad 11: Net-(U1-Pad11) -> /EXT2
- U1 pad 4: Net-(U1-Pad4) -> /CHARGING
- U1 pad 8: Net-(U1-Pad8) -> /EXT3
- U1 pad 9: Net-(U1-Pad9) -> /EXT4
Routing:
- net /IO2: track 73.7 -> 0.00 mm
- net /IO12: track 29.4 -> 0.00 mm
- net Net-(R7-Pad2): track 0.00 -> 28.3 mm, vias 0 -> 2
- net /RX: track 38.8 -> 65.5 mm
- net /IO0: track 5.25 -> 27.0 mm
- net /IO13: track 22.2 -> 0.81 mm
- net +3V3: track 130.7 -> 113.4 mm
- net /IO14: track 16.4 -> 0.00 mm
- net Net-(R10-Pad2): track 14.9 -> 0.00 mm
- net /IO15: track 13.1 -> 0.00 mm
- net /TX: track 43.2 -> 33.2 mm
- net Net-(D5-Pad2): track 0.00 -> 3.44 mm
- net /ONE1: track 0.00 -> 3.14 mm
- net Net-(D5-Pad1): track 0.00 -> 2.54 mm
- net /MCP73831/V_STATUS: track 2.54 -> 0.00 mm
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
Commit message: feat: pcb v1
Parts:
- removed the C10 at (156.7, 69.1)
- removed the D2 at (108.5, 73.5)
- removed the J13 at (111.5, 108.2)
- removed the R10 at (154.2, 82.4)
- removed the R11 at (141.8, 111.3)
- removed the R11 at (133.9, 101.4)
- removed the R7 at (114.2, 77.3)
- removed the R8 at (114.2, 74.8)
- added C2: 10uF, Capacitor_SMD:C_0805_2012Metric_Pad1.15x1.40mm_HandSolder, F.Cu at (156.5, 70.7)
- added J9: IO_RGBW, Connector_PinHeader_2.54mm:PinHeader_1x08_P2.54mm_Vertical, F.Cu at (138.2, 112.4)
- added R3: 4.7k, Resistor_SMD:R_0805_2012Metric_Pad1.15x1.40mm_HandSolder, F.Cu at (142.8, 109.3)
- moved TP6 6.43 mm to (142.8, 102.5), turned to 270 degrees
- moved TP1 4.46 mm to (142.8, 94.1)
- moved R2 1.52 mm to (119.0, 98.0)
- moved D2 1.52 mm to (118.9, 101.2)
- moved TP7 0.38 mm to (90.4, 69.7)
- renumbered C11 to C1, C6 to C10, C7 to C11, C8 to C3, C9 to C4, C1 to C5, C2 to C6, C3 to C7, C4 to C8, C5 to C9, D3 to D1, D4 to D3, D5 to D4, D1 to D5, J2 to J1, J8 to J10, J10 to J11, J11 to J12, J12 to J13, J9 to J14, J3 to J15, J4 to J16, J5 to J17, J1 to J18, J14 to J2, J7 to J3, J6 to J4, J15 to J5, J16 to J6, J17 to J7, J18 to J8, R9 to R1, R6 to R10, R4 to R11, R8 to R2, R7 to R4, R10 to R5, R1 to R6, R5 to R7, R2 to R8, R3 to R9, TP3 to TP1, TP1 to TP2, TP5 to TP3, TP6 to TP4, TP4 to TP5, TP8 to TP6, TP2 to TP8, U4 to U2, U6 to U3, U2 to U4, U3 to U5, U5 to U6
Connections:
- net /ADC renamed ADC
- net /CHARGING renamed CHARGING
Routing:
- net /ONE2: track 0.00 -> 69.1 mm
- net /ONE1: track 3.14 -> 53.5 mm, vias 0 -> 1
- net +3V3: track 113.4 -> 158.8 mm
- net /IO12: track 0.00 -> 43.4 mm, vias 0 -> 2
- net /IO13: track 0.81 -> 42.6 mm, vias 0 -> 2
- net /IO15: track 0.00 -> 39.1 mm, vias 0 -> 2
- net /IO14: track 0.00 -> 38.6 mm, vias 0 -> 2
- net /EXT1: track 0.00 -> 32.8 mm, vias 0 -> 2
- net /EXT3: track 0.00 -> 31.2 mm, vias 0 -> 2
- net +12V: track 134.2 -> 164.7 mm
- net /EXT2: track 0.00 -> 29.7 mm, vias 0 -> 2
- net /EXT4: track 0.00 -> 29.3 mm, vias 0 -> 2
- net CHARGING: track 2.54 -> 31.4 mm, vias 0 -> 2
- net +BATT: track 84.4 -> 108.5 mm
- net ADC: track 5.08 -> 25.2 mm, vias 0 -> 2
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