File: kicad/esp32.sch (KiCad schematic (older format))
At the start: 42 parts, among them J10 Green, J11 Blue, J12 White, J13 IO_RGBW, J14 +12V, J15 hole, J16 hole, J17 hole, J18 hole, J2 5 / 12V, J3 CONN FT232RL, J4 RJ12-I2C, J5 RJ12-I2C, J6 Onewire, J7 Onewire, J8 Red, J9 Pad, Q1 BSP75, Q2 BSP75, Q3 BSP75, Q4 BSP75, SW1 RESET, SW2 PROG, U1 ESP32-WROOM-32U, U4 MS5637, U6 Si7020-A20, U7 DS18B20

Commit message: work in progress
Parts:
- added D2, D5: LED, LED_SMD:LED_0805_2012Metric_Pad1.15x1.40mm_HandSolder, symbol Device:LED
- added R10, R8: 10k, Resistor_SMD:R_0805_2012Metric_Pad1.15x1.40mm_HandSolder, symbol Device:R
- C10: footprint (none) -> Capacitor_SMD:C_0805_2012Metric_Pad1.15x1.40mm_HandSolder
- C11: renamed from C?; footprint (none) -> Capacitor_SMD:C_0805_2012Metric_Pad1.15x1.40mm_HandSolder
- R7: renamed from R?; footprint (none) -> Resistor_SMD:R_0805_2012Metric_Pad1.15x1.40mm_HandSolder
Connections:
- net labels added: IO0
- wire segments 119 -> 125
Other:
- note added: "3.10.2019"
- note added: "ESP-32 playground"
- note removed: "18.01.2019"
- note removed: "ESP-12e playground"
Changed lines of the file:
@@
 EESchema Schematic File Version 4
-LIBS:esp8266-cache
+LIBS:esp32-cache
 EELAYER 29 0
 EELAYER END
@@
 NoConn ~ 1000 3200
 Text Notes 7400 7500 0    50   ~ 0
-ESP-12e playground
+ESP-32 playground
 Text Notes 8150 7650 0    50   ~ 0
-18.01.2019
+3.10.2019
 $Comp
 L power:GND #PWR0120
@@
 F 0 "C10" V 3198 4200 50  0000 C CNN
 F 1 "100nF" V 3289 4200 50  0000 C CNN
-F 2 "" H 3488 4050 50  0001 C CNN
+F 2 "Capacitor_SMD:C_0805_2012Metric_Pad1.15x1.40mm_HandSolder" H 3488 4050 50  0001 C CNN
 F 3 "~" H 3450 4200 50  0001 C CNN
 	1    3450 4200
@@
 $EndComp
 $Comp
-L Device:R R?
+L Device:R R7
 U 1 1 5DB2F657
 P 5500 4050
-F 0 "R?" V 5500 4050 50  0000 C CNN
+F 0 "R7" V 5500 4050 50  0000 C CNN
 F 1 "499" V 5600 4050 50  0000 C CNN
-F 2 "" V 5430 4050 50  0001 C CNN
+F 2 "Resistor_SMD:R_0805_2012Metric_Pad1.15x1.40mm_HandSolder" V 5430 4050 50  0001 C CNN
 F 3 "~" H 5500 4050 50  0001 C CNN
 	1    5500 4050
@@
 TX
 $Comp
-L Device:C C?
+L Device:C C11
 U 1 1 5DB41C5E
 P 5600 3550
-F 0 "C?" V 5348 3550 50  0000 C CNN
+F 0 "C11" V 5348 3550 50  0000 C CNN
 F 1 "100nF" V 5439 3550 50  0000 C CNN
-F 2 "" H 5638 3400 50  0001 C CNN
+F 2 "Capacitor_SMD:C_0805_2012Metric_Pad1.15x1.40mm_HandSolder" H 5638 3400 50  0001 C CNN
 F 3 "~" H 5600 3550 50  0001 C CNN
 	1    5600 3550
@@
 Wire Wire Line
 	5850 3950 5950 3950
+$Comp
+L Device:LED D5
+U 1 1 5DA3D956
+P 5500 5150
+F 0 "D5" H 5493 4895 50  0000 C CNN
+F 1 "LED" H 5493 4986 50  0000 C CNN
+F 2 "LED_SMD:LED_0805_2012Metric_Pad1.15x1.40mm_HandSolder" H 5500 5150 50  0001 C CNN
+F 3 "~" H 5500 5150 50  0001 C CNN
+	1    5500 5150
+	-1   0    0    1
+$EndComp
+$Comp
+L Device:R R10
+U 1 1 5DA4F654
+P 5900 5150
+F 0 "R10" V 5800 5150 50  0000 C CNN
+F 1 "10k" V 5900 5150 50  0000 C CNN
+F 2 "Resistor_SMD:R_0805_2012Metric_Pad1.15x1.40mm_HandSolder" V 5830 5150 50  0001 C CNN
+F 3 "~" H 5900 5150 50  0001 C CNN
+	1    5900 5150
+	0    1    1    0
+$EndComp
+$Comp
+L power:GND #PWR0112
+U 1 1 5DA50594
+P 6200 5150
+F 0 "#PWR0112" H 6200 4900 50  0001 C CNN
+F 1 "GND" H 6205 4977 50  0000 C CNN
+F 2 "" H 6200 5150 50  0001 C CNN
+F 3 "" H 6200 5150 50  0001 C CNN
+	1    6200 5150
+	1    0    0    -1
+$EndComp
+Wire Wire Line
+	5200 5150 5350 5150
+Wire Wire Line
+	5650 5150 5750 5150
+Wire Wire Line
+	6050 5150 6200 5150
+$Comp
+L Device:LED D2
+U 1 1 5DA6B048
+P 7550 1650
+F 0 "D2" H 7543 1395 50  0000 C CNN
+F 1 "LED" H 7543 1486 50  0000 C CNN
+F 2 "LED_SMD:LED_0805_2012Metric_Pad1.15x1.40mm_HandSolder" H 7550 1650 50  0001 C CNN
+F 3 "~" H 7550 1650 50  0001 C CNN
+	1    7550 1650
+	-1   0    0    1
+$EndComp
+$Comp
+L Device:R R8
+U 1 1 5DA6C56C
+P 7950 1650
+F 0 "R8" V 7850 1650 50  0000 C CNN
+F 1 "10k" V 7950 1650 50  0000 C CNN
+F 2 "Resistor_SMD:R_0805_2012Metric_Pad1.15x1.40mm_HandSolder" V 7880 1650 50  0001 C CNN
+F 3 "~" H 7950 1650 50  0001 C CNN
+	1    7950 1650
+	0    1    1    0
+$EndComp
+$Comp
+L power:GND #PWR0118
+U 1 1 5DA6DCAD
+P 8200 1650
+F 0 "#PWR0118" H 8200 1400 50  0001 C CNN
+F 1 "GND" H 8205 1477 50  0000 C CNN
+F 2 "" H 8200 1650 50  0001 C CNN
+F 3 "" H 8200 1650 50  0001 C CNN
+	1    8200 1650
+	1    0    0    -1
+$EndComp
+Wire Wire Line
+	8100 1650 8200 1650
+Wire Wire Line
+	7800 1650 7700 1650
+Wire Wire Line
+	7400 1650 7250 1650
+Connection ~ 7250 1650
+Text Label 5200 3950 0    50   ~ 0
+IO0
 $EndSCHEMATC

Commit message: chore: working on pcb
Parts:
- removed U7: DS18B20, Package_TO_SOT_THT:TO-92_Inline, symbol Sensor_Temperature:DS18B20
- added R11: 4.7k, Resistor_SMD:R_0805_2012Metric_Pad1.15x1.40mm_HandSolder, symbol Device:R
- added TP8: OneWire, TestPoint:TestPoint_2Pads_Pitch2.54mm_Drill0.8mm, symbol Connector:TestPoint_2Pole
- C10: value 100nF -> 10uF
Connections:
- net labels added: CHARGING, EXT1, EXT2, EXT3, EXT4
- net labels removed: IO2, IO34, IO35
- wire segments 125 -> 133
Changed lines of the file:
@@
 L Switch:SW_Push SW1
 U 1 1 5C3B7657
-P 3450 3950
-F 0 "SW1" H 3450 4235 50  0000 C CNN
-F 1 "RESET" H 3450 4144 50  0000 C CNN
-F 2 "Button_Switch_SMD:SW_SPST_PTS645" H 3450 4150 50  0001 C CNN
-F 3 "" H 3450 4150 50  0001 C CNN
-	1    3450 3950
+P 3050 3950
+F 0 "SW1" H 3050 4235 50  0000 C CNN
+F 1 "RESET" H 3050 4144 50  0000 C CNN
+F 2 "Button_Switch_SMD:SW_SPST_PTS645" H 3050 4150 50  0001 C CNN
+F 3 "" H 3050 4150 50  0001 C CNN
+	1    3050 3950
 	1    0    0    -1
 $EndComp
@@
 L power:GND #PWR0119
 U 1 1 5C3B85F9
-P 3100 3950
-F 0 "#PWR0119" H 3100 3700 50  0001 C CNN
-F 1 "GND" H 3105 3777 50  0000 C CNN
-F 2 "" H 3100 3950 50  0001 C CNN
-F 3 "" H 3100 3950 50  0001 C CNN
-	1    3100 3950
-	1    0    0    -1
-$EndComp
-Wire Wire Line
-	3100 3950 3250 3950
-Wire Wire Line
-	3650 3950 3850 3950
-Connection ~ 3850 3950
-Wire Wire Line
-	3850 3900 3850 3950
+P 2700 3950
+F 0 "#PWR0119" H 2700 3700 50  0001 C CNN
+F 1 "GND" H 2705 3777 50  0000 C CNN
+F 2 "" H 2700 3950 50  0001 C CNN
+F 3 "" H 2700 3950 50  0001 C CNN
+	1    2700 3950
+	1    0    0    -1
+$EndComp
+Wire Wire Line
+	2700 3950 2850 3950
+Wire Wire Line
+	3250 3950 3450 3950
+Connection ~ 3450 3950
+Wire Wire Line
+	3450 3900 3450 3950
 $Comp
 L rj12:RJ12-I2C J4
@@
 L Device:R R9
 U 1 1 5C3BB3E1
-P 9000 1550
-F 0 "R9" H 9070 1596 50  0000 L CNN
-F 1 "4.7k" H 9070 1505 50  0000 L CNN
-F 2 "Resistor_SMD:R_0805_2012Metric_Pad1.15x1.40mm_HandSolder" V 8930 1550 50  0001 C CNN
-F 3 "~" H 9000 1550 50  0001 C CNN
-	1    9000 1550
+P 8900 1100
+F 0 "R9" H 8970 1146 50  0000 L CNN
+F 1 "4.7k" H 8970 1055 50  0000 L CNN
+F 2 "Resistor_SMD:R_0805_2012Metric_Pad1.15x1.40mm_HandSolder" V 8830 1100 50  0001 C CNN
+F 3 "~" H 8900 1100 50  0001 C CNN
+	1    8900 1100
 	1    0    0    -1
 $EndComp
@@
 L power:+3.3V #PWR0114
 U 1 1 5C3BB43D
-P 9000 1250
-F 0 "#PWR0114" H 9000 1100 50  0001 C CNN
-F 1 "+3.3V" H 9015 1423 50  0000 C CNN
-F 2 "" H 9000 1250 50  0001 C CNN
-F 3 "" H 9000 1250 50  0001 C CNN
-	1    9000 1250
-	1    0    0    -1
-$EndComp
-Wire Wire Line
-	8650 1700 9000 1700
-Wire Wire Line
-	9000 1700 9150 1700
-Connection ~ 9000 1700
-Wire Wire Line
-	9000 1250 9000 1400
-Text Label 8650 1700 0    50   ~ 0
-IO2
+P 8900 800
+F 0 "#PWR0114" H 8900 650 50  0001 C CNN
+F 1 "+3.3V" H 8915 973 50  0000 C CNN
+F 2 "" H 8900 800 50  0001 C CNN
+F 3 "" H 8900 800 50  0001 C CNN
+	1    8900 800
+	1    0    0    -1
+$EndComp
+Wire Wire Line
+	8550 1250 8900 1250
+Wire Wire Line
+	8900 1250 9050 1250
+Connection ~ 8900 1250
+Wire Wire Line
+	8900 800  8900 950
+Text Label 8550 1250 0    50   ~ 0
+ONE1
 Text Label 4750 2250 0    50   ~ 0
 ADC
@@
 Text Label 2250 1950 0    50   ~ 0
 VCC_FTDI
-Text Label 3700 3950 0    50   ~ 0
+Text Label 3300 3950 0    50   ~ 0
 RST
 $Sheet
@@
 $EndComp
 $Comp
-L Sensor_Temperature:DS18B20 U7
-U 1 1 5C3F9182
-P 10050 2700
-F 0 "U7" H 9820 2746 50  0000 R CNN
-F 1 "DS18B20" H 9820 2655 50  0000 R CNN
-F 2 "Package_TO_SOT_THT:TO-92_Inline" H 9050 2450 50  0001 C CNN
-F 3 "http://datasheets.maximintegrated.com/en/ds/DS18B20.pdf" H 9900 2950 50  0001 C CNN
-	1    10050 2700
-	1    0    0    -1
-$EndComp
-$Comp
 L power:GND #PWR0132
 U 1 1 5C3FE6C9
@@
 L Connector:TestPoint_2Pole TP3
 U 1 1 5C4381A5
-P 9150 1900
-F 0 "TP3" V 9104 1958 50  0000 L CNN
-F 1 "OneWire" V 9195 1958 50  0000 L CNN
-F 2 "TestPoint:TestPoint_2Pads_Pitch2.54mm_Drill0.8mm" H 9150 1900 50  0001 C CNN
-F 3 "~" H 9150 1900 50  0001 C CNN
-	1    9150 1900
+P 9050 1450
+F 0 "TP3" V 9004 1508 50  0000 L CNN
+F 1 "OneWire" V 9095 1508 50  0000 L CNN
+F 2 "TestPoint:TestPoint_2Pads_Pitch2.54mm_Drill0.8mm" H 9050 1450 50  0001 C CNN
+F 3 "~" H 9050 1450 50  0001 C CNN
+	1    9050 1450
 	0    1    1    0
 $EndComp
-Connection ~ 9150 1700
-Wire Wire Line
-	9150 1700 9300 1700
-$Comp
-L power:GND #PWR0140
-U 1 1 5C438384
-P 9150 2200
-F 0 "#PWR0140" H 9150 1950 50  0001 C CNN
-F 1 "GND" H 9155 2027 50  0000 C CNN
-F 2 "" H 9150 2200 50  0001 C CNN
-F 3 "" H 9150 2200 50  0001 C CNN
-	1    9150 2200
-	1    0    0    -1
-$EndComp
-Wire Wire Line
-	9150 2200 9150 2100
+Connection ~ 9050 1250
+Wire Wire Line
+	9050 1250 9200 1250
 $Comp
 L Connector:Conn_01x08_Female J13
@@
 	6250 3250 6450 3250
 Text Label 6250 3550 0    50   ~ 0
-IO15
+EXT4
 Text Label 6250 3450 0    50   ~ 0
-IO14
+EXT3
 Text Label 6250 3350 0    50   ~ 0
-IO13
+EXT2
 Text Label 6250 3250 0    50   ~ 0
-IO12
+EXT1
 Wire Wire Line
 	6450 2950 6350 2950
@@
 SDA
 $Comp
-L power:GND #PWR0158
-U 1 1 5C4B9B38
-P 10050 3100
-F 0 "#PWR0158" H 10050 2850 50  0001 C CNN
-F 1 "GND" H 10055 2927 50  0000 C CNN
-F 2 "" H 10050 3100 50  0001 C CNN
-F 3 "" H 10050 3100 50  0001 C CNN
-	1    10050 3100
-	1    0    0    -1
-$EndComp
-$Comp
-L power:+3.3V #PWR0159
-U 1 1 5C4B9C10
-P 10050 2300
-F 0 "#PWR0159" H 10050 2150 50  0001 C CNN
-F 1 "+3.3V" H 10065 2473 50  0000 C CNN
-F 2 "" H 10050 2300 50  0001 C CNN
-F 3 "" H 10050 2300 50  0001 C CNN
-	1    10050 2300
-	1    0    0    -1
-$EndComp
-Wire Wire Line
-	10050 2400 10050 2300
-Wire Wire Line
-	10050 3000 10050 3100
-Wire Wire Line
-	10350 2700 10650 2700
-Text Label 10450 2700 0    50   ~ 0
-IO2
-$Comp
 L Test_points:Test_i2C TP2
 U 1 1 5C4D4A7A
@@
 	10250 1800 10500 1800
 Text Label 10300 1150 0    50   ~ 0
-IO34
+ONE1
 Text Label 10300 1800 0    50   ~ 0
-IO35
+ONE2
 Text Label 5250 6250 0    50   ~ 0
 ONE2
@@
 L Device:C C10
 U 1 1 5DAACE54
-P 3450 4200
-F 0 "C10" V 3198 4200 50  0000 C CNN
-F 1 "100nF" V 3289 4200 50  0000 C CNN
-F 2 "Capacitor_SMD:C_0805_2012Metric_Pad1.15x1.40mm_HandSolder" H 3488 4050 50  0001 C CNN
-F 3 "~" H 3450 4200 50  0001 C CNN
-	1    3450 4200
+P 3050 4200
+F 0 "C10" V 2798 4200 50  0000 C CNN
+F 1 "10uF" V 2889 4200 50  0000 C CNN
+F 2 "Capacitor_SMD:C_0805_2012Metric_Pad1.15x1.40mm_HandSolder" H 3088 4050 50  0001 C CNN
+F 3 "~" H 3050 4200 50  0001 C CNN
+	1    3050 4200
 	0    1    1    0
 $EndComp
 Wire Wire Line
-	3250 3950 3250 4200
-Wire Wire Line
-	3250 4200 3300 4200
-Connection ~ 3250 3950
-Wire Wire Line
-	3600 4200 3850 4200
-Wire Wire Line
-	3850 4200 3850 3950
+	2850 3950 2850 4200
+Wire Wire Line
+	2850 4200 2900 4200
+Connection ~ 2850 3950
+Wire Wire Line
+	3200 4200 3450 4200
+Wire Wire Line
+	3450 4200 3450 3950
 Wire Wire Line
 	5200 5850 5500 5850
@@
 Wire Wire Line
 	5800 3950 5850 3950
-Wire Wire Line
-	3850 3950 4000 3950
 $Comp
 L RF_Module:ESP32-WROOM-32U U1
@@
 Text Label 5200 3950 0    50   ~ 0
 IO0
+Wire Wire Line
+	4700 2050 4950 2050
+Text Label 4750 2050 0    50   ~ 0
+CHARGING
+Wire Wire Line
+	3450 3950 4000 3950
+Wire Wire Line
+	4000 4150 3650 4150
+Text Label 3650 4150 0    50   ~ 0
+CHARGING
+Wire Wire Line
+	5200 5950 5500 5950
+Wire Wire Line
+	5200 6050 5500 6050
+Wire Wire Line
+	5200 5750 5500 5750
+Wire Wire Line
+	5200 5650 5500 5650
+Text Label 5250 5950 0    50   ~ 0
+EXT3
+Text Label 5250 6050 0    50   ~ 0
+EXT4
+Text Label 5250 5650 0    50   ~ 0
+EXT1
+Text Label 5250 5750 0    50   ~ 0
+EXT2
+Wire Wire Line
+	9050 1750 9050 1650
+$Comp
+L power:GND #PWR0140
+U 1 1 5C438384
+P 9050 1750
+F 0 "#PWR0140" H 9050 1500 50  0001 C CNN
+F 1 "GND" H 9055 1577 50  0000 C CNN
+F 2 "" H 9050 1750 50  0001 C CNN
+F 3 "" H 9050 1750 50  0001 C CNN
+	1    9050 1750
+	1    0    0    -1
+$EndComp
+$Comp
+L Device:R R11
+U 1 1 5DB53745
+P 8850 2450
+F 0 "R11" H 8920 2496 50  0000 L CNN
+F 1 "4.7k" H 8920 2405 50  0000 L CNN
+F 2 "Resistor_SMD:R_0805_2012Metric_Pad1.15x1.40mm_HandSolder" V 8780 2450 50  0001 C CNN
+F 3 "~" H 8850 2450 50  0001 C CNN
+	1    8850 2450
+	1    0    0    -1
+$EndComp
+$Comp
+L power:+3.3V #PWR0124
+U 1 1 5DB5374F
+P 8850 2150
+F 0 "#PWR0124" H 8850 2000 50  0001 C CNN
+F 1 "+3.3V" H 8865 2323 50  0000 C CNN
+F 2 "" H 8850 2150 50  0001 C CNN
+F 3 "" H 8850 2150 50  0001 C CNN
+	1    8850 2150
+	1    0    0    -1
+$EndComp
+Wire Wire Line
+	8500 2600 8850 2600
+Wire Wire Line
+	8850 2600 9000 2600
+Connection ~ 8850 2600
+Wire Wire Line
+	8850 2150 8850 2300
+Text Label 8500 2600 0    50   ~ 0
+ONE2
+$Comp
+L Connector:TestPoint_2Pole TP8
+U 1 1 5DB5375E
+P 9000 2800
+F 0 "TP8" V 8954 2858 50  0000 L CNN
+F 1 "OneWire" V 9045 2858 50  0000 L CNN
+F 2 "TestPoint:TestPoint_2Pads_Pitch2.54mm_Drill0.8mm" H 9000 2800 50  0001 C CNN
+F 3 "~" H 9000 2800 50  0001 C CNN
+	1    9000 2800
+	0    1    1    0
+$EndComp
+Connection ~ 9000 2600
+Wire Wire Line
+	9000 2600 9150 2600
+Wire Wire Line
+	9000 3100 9000 3000
+$Comp
+L power:GND #PWR0167
+U 1 1 5DB5376B
+P 9000 3100
+F 0 "#PWR0167" H 9000 2850 50  0001 C CNN
+F 1 "GND" H 9005 2927 50  0000 C CNN
+F 2 "" H 9000 3100 50  0001 C CNN
+F 3 "" H 9000 3100 50  0001 C CNN
+	1    9000 3100
+	1    0    0    -1
+$EndComp
 $EndSCHEMATC

Commit message: feat: pcb v1
Parts:
- renumbered C11 to C1, C10 to C2, C8 to C3, C9 to C4, D3 to D1, D4 to D3, D5 to D4, J2 to J1, J8 to J10, J10 to J11, J11 to J12, J12 to J13, J9 to J14, J3 to J15, J4 to J16, J5 to J17, J14 to J2, J7 to J3, J6 to J4, J15 to J5, J16 to J6, J17 to J7, J18 to J8, J13 to J9, R9 to R1, R8 to R2, R11 to R3, R7 to R4, R10 to R5, TP3 to TP1, TP1 to TP2, TP5 to TP3, TP6 to TP4, TP4 to TP5, TP8 to TP6, TP2 to TP8, U4 to U2, U6 to U3
