File: kicad/esp32.sch (KiCad schematic (older format))
At the start: 46 parts, among them J1 5 / 12V, J10 Red, J11 Green, J12 Blue, J13 White, J14 Pad, J15 CONN FT232RL, J16 RJ12-I2C, J17 RJ12-I2C, J2 +12V, J3 Onewire, J4 Onewire, J5 hole, J6 hole, J7 hole, J8 hole, J9 IO_RGBW, Q1 BSP75, Q2 BSP75, Q3 BSP75, Q4 BSP75, SW1 RESET, SW2 PROG, U1 ESP32-WROOM-32U, U2 MS5637, U3 Si7020-A20

Commit message: fix: pullup on reset close: https://github.com/Hackuarium/esp-32wroom/issues/1
Parts:
- added R16: 10k, Resistor_SMD:R_0805_2012Metric_Pad1.15x1.40mm_HandSolder, symbol Device:R
Connections:
- wire segments 130 -> 133
Changed lines of the file:
@@
 IO0
 Wire Wire Line
-	3450 3950 4000 3950
+	3450 3950 3800 3950
 Wire Wire Line
 	5200 5950 5500 5950
@@
 Wire Wire Line
 	700  1650 950  1650
+$Comp
+L Device:R R16
+U 1 1 5DF1C5AB
+P 3800 3700
+F 0 "R16" H 3870 3746 50  0000 L CNN
+F 1 "10k" H 3870 3655 50  0000 L CNN
+F 2 "Resistor_SMD:R_0805_2012Metric_Pad1.15x1.40mm_HandSolder" V 3730 3700 50  0001 C CNN
+F 3 "~" H 3800 3700 50  0001 C CNN
+	1    3800 3700
+	1    0    0    -1
+$EndComp
+$Comp
+L power:+3.3V #PWR0119
+U 1 1 5DF1CCF5
+P 3800 3450
+F 0 "#PWR0119" H 3800 3300 50  0001 C CNN
+F 1 "+3.3V" H 3815 3623 50  0000 C CNN
+F 2 "" H 3800 3450 50  0001 C CNN
+F 3 "" H 3800 3450 50  0001 C CNN
+	1    3800 3450
+	1    0    0    -1
+$EndComp
+Wire Wire Line
+	3800 3450 3800 3550
+Wire Wire Line
+	3800 3850 3800 3950
+Connection ~ 3800 3950
+Wire Wire Line
+	3800 3950 4000 3950
 $EndSCHEMATC

Commit message: feat: add light and temperature sensors. closes https://github.com/Hackuarium/esp-32wroom/issues/6 and https://github.com/Hackuarium/esp-32wroom/issues/5
Parts:
- added R17: 4.7k, Resistor_SMD:R_0805_2012Metric_Pad1.15x1.40mm_HandSolder, symbol Device:R
- added U7: DS18B20U, Package_SO:MSOP-8_3x3mm_P0.65mm, symbol Sensor_Temperature:DS18B20U
- added U8: TCS3400, OptoDevice:Broadcom_DFN-6_2x2mm_P0.65mm, symbol TCS3400:TCS3400
Connections:
- net labels added: ONE3
- wire segments 133 -> 144
Changed lines of the file:
@@
 L Test_points:Test_i2C TP8
 U 1 1 5C4D4A7A
-P 7100 5650
-F 0 "TP8" H 7016 5975 50  0000 C CNN
-F 1 "Test_i2C" H 7016 5884 50  0000 C CNN
-F 2 "Connector_PinHeader_2.54mm:PinHeader_1x03_P2.54mm_Vertical" H 7150 5850 50  0001 C CNN
-F 3 "~" H 7150 5850 50  0001 C CNN
-	1    7100 5650
+P 6450 6450
+F 0 "TP8" H 6366 6775 50  0000 C CNN
+F 1 "Test_i2C" H 6366 6684 50  0000 C CNN
+F 2 "Connector_PinHeader_2.54mm:PinHeader_1x03_P2.54mm_Vertical" H 6500 6650 50  0001 C CNN
+F 3 "~" H 6500 6650 50  0001 C CNN
+	1    6450 6450
 	1    0    0    -1
 $EndComp
@@
 L power:GND #PWR038
 U 1 1 5C4D4B30
-P 7300 5750
-F 0 "#PWR038" H 7300 5500 50  0001 C CNN
-F 1 "GND" H 7305 5577 50  0000 C CNN
-F 2 "" H 7300 5750 50  0001 C CNN
-F 3 "" H 7300 5750 50  0001 C CNN
-	1    7300 5750
-	1    0    0    -1
-$EndComp
-Wire Wire Line
-	7300 5750 7150 5750
-Wire Wire Line
-	7150 5650 7300 5650
-Wire Wire Line
-	7150 5550 7300 5550
-Text Label 7300 5550 0    50   ~ 0
+P 6650 6550
+F 0 "#PWR038" H 6650 6300 50  0001 C CNN
+F 1 "GND" H 6655 6377 50  0000 C CNN
+F 2 "" H 6650 6550 50  0001 C CNN
+F 3 "" H 6650 6550 50  0001 C CNN
+	1    6650 6550
+	1    0    0    -1
+$EndComp
+Wire Wire Line
+	6650 6550 6500 6550
+Wire Wire Line
+	6500 6450 6650 6450
+Wire Wire Line
+	6500 6350 6650 6350
+Text Label 6650 6350 0    50   ~ 0
 SCL
-Text Label 7300 5650 0    50   ~ 0
+Text Label 6650 6450 0    50   ~ 0
 SDA
 $Comp
@@
 Wire Wire Line
 	3800 3950 4000 3950
+$Comp
+L Sensor_Temperature:DS18B20U U7
+U 1 1 5DF3B94D
+P 10400 2650
+F 0 "U7" H 10056 2696 50  0000 R CNN
+F 1 "DS18B20U" H 10056 2605 50  0000 R CNN
+F 2 "Package_SO:MSOP-8_3x3mm_P0.65mm" H 9450 2400 50  0001 C CNN
+F 3 "http://datasheets.maximintegrated.com/en/ds/DS18B20.pdf" H 10250 2900 50  0001 C CNN
+	1    10400 2650
+	1    0    0    -1
+$EndComp
+Text GLabel 10950 2650 2    50   Input ~ 0
+ONE3
+Wire Wire Line
+	10700 2650 10800 2650
+$Comp
+L power:GND #PWR0120
+U 1 1 5DF44B6D
+P 10400 3100
+F 0 "#PWR0120" H 10400 2850 50  0001 C CNN
+F 1 "GND" H 10405 2927 50  0000 C CNN
+F 2 "" H 10400 3100 50  0001 C CNN
+F 3 "" H 10400 3100 50  0001 C CNN
+	1    10400 3100
+	1    0    0    -1
+$EndComp
+$Comp
+L power:+3.3V #PWR0121
+U 1 1 5DF44FD5
+P 10400 2250
+F 0 "#PWR0121" H 10400 2100 50  0001 C CNN
+F 1 "+3.3V" H 10415 2423 50  0000 C CNN
+F 2 "" H 10400 2250 50  0001 C CNN
+F 3 "" H 10400 2250 50  0001 C CNN
+	1    10400 2250
+	1    0    0    -1
+$EndComp
+Wire Wire Line
+	10400 2250 10400 2350
+Wire Wire Line
+	10400 2950 10400 3100
+$Comp
+L Device:R R17
+U 1 1 5DF53837
+P 10800 2400
+F 0 "R17" H 10870 2446 50  0000 L CNN
+F 1 "4.7k" H 10870 2355 50  0000 L CNN
+F 2 "Resistor_SMD:R_0805_2012Metric_Pad1.15x1.40mm_HandSolder" V 10730 2400 50  0001 C CNN
+F 3 "~" H 10800 2400 50  0001 C CNN
+	1    10800 2400
+	1    0    0    -1
+$EndComp
+Wire Wire Line
+	10800 2650 10800 2550
+Connection ~ 10800 2650
+Wire Wire Line
+	10800 2650 10950 2650
+$Comp
+L power:+3.3V #PWR0122
+U 1 1 5DF5B43F
+P 10800 2200
+F 0 "#PWR0122" H 10800 2050 50  0001 C CNN
+F 1 "+3.3V" H 10815 2373 50  0000 C CNN
+F 2 "" H 10800 2200 50  0001 C CNN
+F 3 "" H 10800 2200 50  0001 C CNN
+	1    10800 2200
+	1    0    0    -1
+$EndComp
+Wire Wire Line
+	10800 2200 10800 2250
+Text GLabel 5600 4350 2    50   Input ~ 0
+ONE3
+Wire Wire Line
+	5200 4350 5600 4350
+$Comp
+L TCS3400:TCS3400 U8
+U 1 1 5DF7E3BD
+P 7000 5600
+F 0 "U8" H 7000 6115 50  0000 C CNN
+F 1 "TCS3400" H 7000 6024 50  0000 C CNN
+F 2 "OptoDevice:Broadcom_DFN-6_2x2mm_P0.65mm" H 7000 5650 50  0001 C CNN
+F 3 "" H 7000 5650 50  0001 C CNN
+	1    7000 5600
+	1    0    0    -1
+$EndComp
+$Comp
+L power:+3.3V #PWR?
+U 1 1 5DF9ED5F
+P 6600 5450
+F 0 "#PWR?" H 6600 5300 50  0001 C CNN
+F 1 "+3.3V" H 6615 5623 50  0000 C CNN
+F 2 "" H 6600 5450 50  0001 C CNN
+F 3 "" H 6600 5450 50  0001 C CNN
+	1    6600 5450
+	1    0    0    -1
+$EndComp
+$Comp
+L power:GND #PWR?
+U 1 1 5DF9F4DA
+P 6600 5750
+F 0 "#PWR?" H 6600 5500 50  0001 C CNN
+F 1 "GND" H 6605 5577 50  0000 C CNN
+F 2 "" H 6600 5750 50  0001 C CNN
+F 3 "" H 6600 5750 50  0001 C CNN
+	1    6600 5750
+	1    0    0    -1
+$EndComp
+Wire Wire Line
+	6600 5750 6700 5750
+Wire Wire Line
+	6700 5450 6600 5450
+Text GLabel 6550 5600 0    50   Input ~ 0
+SCL
+Text GLabel 7450 5750 2    50   Input ~ 0
+SDA
+Wire Wire Line
+	6550 5600 6700 5600
+Wire Wire Line
+	7300 5750 7450 5750
 $EndSCHEMATC

Commit message: fix: not connected pins
Connections:
- wire segments 144 -> 146
- no-connect marks 12 -> 26
Changed lines of the file:
@@
-$EndComp
-$Comp
-L Sensor_Humidity:Si7020-A20 U3
-U 1 1 5C3A5AF4
-P 10150 5600
-F 0 "U3" H 10591 5646 50  0000 L CNN
-F 1 "Si7020-A20" H 10591 5555 50  0000 L CNN
-F 2 "Package_DFN_QFN:DFN-6-1EP_3x3mm_P1mm_EP1.5x2.4mm" H 10150 5200 50  0001 C CNN
-F 3 "" H 10150 5600 50  0001 C CNN
-	1    10150 5600
-	1    0    0    -1
 $EndComp
 $Comp
@@
 RST
 $Comp
-L power:GND #PWR08
-U 1 1 5C3D4B6C
-P 10600 1600
-F 0 "#PWR08" H 10600 1350 50  0001 C CNN
-F 1 "GND" H 10605 1427 50  0000 C CNN
-F 2 "" H 10600 1600 50  0001 C CNN
-F 3 "" H 10600 1600 50  0001 C CNN
-	1    10600 1600
-	1    0    0    -1
-$EndComp
-$Comp
 L power:+3.3V #PWR07
 U 1 1 5C3D5BDB
@@
 Wire Wire Line
 	10250 1500 10600 1500
-Wire Wire Line
-	10600 1600 10250 1600
 $Comp
 L Onewire:Onewire J4
@@
 L power:GND #PWR06
 U 1 1 5C3EE93A
-P 10600 950
-F 0 "#PWR06" H 10600 700 50  0001 C CNN
-F 1 "GND" H 10605 777 50  0000 C CNN
-F 2 "" H 10600 950 50  0001 C CNN
-F 3 "" H 10600 950 50  0001 C CNN
-	1    10600 950
+P 10850 1000
+F 0 "#PWR06" H 10850 750 50  0001 C CNN
+F 1 "GND" H 10950 1000 50  0000 C CNN
+F 2 "" H 10850 1000 50  0001 C CNN
+F 3 "" H 10850 1000 50  0001 C CNN
+	1    10850 1000
 	1    0    0    -1
 $EndComp
@@
 Wire Wire Line
 	10250 850  10600 850
-Wire Wire Line
-	10600 950  10250 950
 Wire Wire Line
 	10250 1150 10500 1150
@@
 $EndComp
 Wire Wire Line
-	10150 5300 10150 5150
-Wire Wire Line
 	10050 5900 10050 6050
 $Comp
@@
 F 3 "" H 10050 6050 50  0001 C CNN
 	1    10050 6050
-	1    0    0    -1
-$EndComp
-$Comp
-L power:+3.3V #PWR034
-U 1 1 5C4375BD
-P 10150 5150
-F 0 "#PWR034" H 10150 5000 50  0001 C CNN
-F 1 "+3.3V" H 10165 5323 50  0000 C CNN
-F 2 "" H 10150 5150 50  0001 C CNN
-F 3 "" H 10150 5150 50  0001 C CNN
-	1    10150 5150
 	1    0    0    -1
 $EndComp
@@
 $EndComp
 $Comp
-L power:+3.3V #PWR?
+L power:+3.3V #PWR0123
 U 1 1 5DF9ED5F
 P 6600 5450
-F 0 "#PWR?" H 6600 5300 50  0001 C CNN
+F 0 "#PWR0123" H 6600 5300 50  0001 C CNN
 F 1 "+3.3V" H 6615 5623 50  0000 C CNN
 F 2 "" H 6600 5450 50  0001 C CNN
@@
 $EndComp
 $Comp
-L power:GND #PWR?
+L power:GND #PWR0124
 U 1 1 5DF9F4DA
 P 6600 5750
-F 0 "#PWR?" H 6600 5500 50  0001 C CNN
+F 0 "#PWR0124" H 6600 5500 50  0001 C CNN
 F 1 "GND" H 6605 5577 50  0000 C CNN
 F 2 "" H 6600 5750 50  0001 C CNN
@@
 Wire Wire Line
 	7300 5750 7450 5750
+NoConn ~ 7300 5600
+NoConn ~ 7300 5450
+NoConn ~ 5200 5550
+NoConn ~ 5200 5250
+NoConn ~ 4000 5150
+NoConn ~ 4000 5250
+NoConn ~ 4000 5350
+NoConn ~ 4000 5450
+NoConn ~ 4000 5550
+NoConn ~ 4000 5650
+NoConn ~ 4000 4250
+NoConn ~ 5200 4450
+NoConn ~ 5200 4950
+NoConn ~ 5200 5050
+Text GLabel 5500 6150 2    50   Input ~ 0
+ONE1
+Text GLabel 5500 6250 2    50   Input ~ 0
+ONE2
+Text Label 5300 4350 0    50   ~ 0
+ONE1
+Text GLabel 5550 5350 2    50   Input ~ 0
+SDA
+Text GLabel 5550 5450 2    50   Input ~ 0
+SCL
+Text GLabel 10500 1150 2    50   Input ~ 0
+ONE1
+Text GLabel 10500 1800 2    50   Input ~ 0
+ONE2
+$Comp
+L power:GND #PWR08
+U 1 1 5C3D4B6C
+P 10850 1650
+F 0 "#PWR08" H 10850 1400 50  0001 C CNN
+F 1 "GND" H 10950 1650 50  0000 C CNN
+F 2 "" H 10850 1650 50  0001 C CNN
+F 3 "" H 10850 1650 50  0001 C CNN
+	1    10850 1650
+	1    0    0    -1
+$EndComp
+Wire Wire Line
+	10850 1650 10850 1600
+Wire Wire Line
+	10250 1600 10850 1600
+Wire Wire Line
+	10850 950  10850 1000
+Wire Wire Line
+	10250 950  10850 950
+Text GLabel 9150 2600 2    50   Input ~ 0
+ONE2
+Text GLabel 9200 1250 2    50   Input ~ 0
+ONE1
+$Comp
+L Sensor_Humidity:Si7020-A20 U3
+U 1 1 5C3A5AF4
+P 10150 5600
+F 0 "U3" H 10591 5646 50  0000 L CNN
+F 1 "Si7020-A20" H 10591 5555 50  0000 L CNN
+F 2 "Package_DFN_QFN:DFN-6-1EP_3x3mm_P1mm_EP1.5x2.4mm" H 10150 5200 50  0001 C CNN
+F 3 "" H 10150 5600 50  0001 C CNN
+	1    10150 5600
+	1    0    0    -1
+$EndComp
+$Comp
+L power:+3.3V #PWR034
+U 1 1 5C4375BD
+P 10150 5150
+F 0 "#PWR034" H 10150 5000 50  0001 C CNN
+F 1 "+3.3V" H 10165 5323 50  0000 C CNN
+F 2 "" H 10150 5150 50  0001 C CNN
+F 3 "" H 10150 5150 50  0001 C CNN
+	1    10150 5150
+	1    0    0    -1
+$EndComp
+Wire Wire Line
+	10150 5150 10150 5300
 $EndSCHEMATC
