File: kicad-rgb/esp32.sch (KiCad schematic (older format))
At the start: 59 parts, among them J1 5 / 12V, J10 R1, J11 G1, J12 B1, J13 W1, J14 GND1, J15 CONN FT232RL, J16 B2, J17 W2, J18 GND2, J19 R3, J20 G3, J21 B3, J22 W3, J23 GND3, J24 R4, J25 G4, J26 B4, J27 GND4, J3 R2, J4 W1, J5 hole, J6 hole, J7 hole, J8 hole, J9 G2, Q1 BSP75, Q10 BSP75, Q11 BSP75, Q12 BSP75, Q13 BSP75, Q14 BSP75, Q15 BSP75, Q16 BSP75, Q2 BSP75, Q3 BSP75, Q4 BSP75, Q5 BSP75, Q6 BSP75, Q7 BSP75, Q8 BSP75, Q9 BSP75, SW1 RESET, SW2 PROG, U1 ESP32-WROOM-32U, U2 DS18B20, U3 PCA9685PW

Commit message: chore: working on kicad-rgb
Parts:
- removed TP2: 5V, TestPoint:TestPoint_2Pads_Pitch2.54mm_Drill0.8mm, symbol Connector:TestPoint_2Pole
Connections:
- wire segments 134 -> 130
Changed lines of the file:
@@
 $Descr A4 11693 8268
 encoding utf-8
-Sheet 1 3
+Sheet 1 1
 Title ""
 Date ""
@@
 Comment4 ""
 $EndDescr
-$Sheet
-S 800  2750 950  550
-U 5C3A2732
-F0 "MCP1703-33" 50
-F1 "schemas/MCP1703-33.sch" 50
-F2 "VDD" I L 800 3000 50
-F3 "3.3V" O R 1750 3000 50
-$EndSheet
 $Comp
 L BSP75:BSP75 Q1
@@
 Wire Wire Line
 	4200 2000 4200 2150
-Wire Wire Line
-	1750 3000 2050 3000
 $Comp
 L power:+3.3V #PWR010
@@
 Text Label 1600 4700 0    50   ~ 0
 RST
-$Sheet
-S 850  1400 950  550
-U 5C3D1997
-F0 "MCP1703-50" 50
-F1 "schemas/MCP1703-50.sch" 50
-F2 "VDD" I L 850 1650 50
-F3 "5.0V" O R 1800 1650 50
-$EndSheet
 $Comp
 L power:GND #PWR027
@@
 	0    1    1    0
 $EndComp
-$Comp
-L Connector:TestPoint_2Pole TP2
-U 1 1 5C44FC41
-P 1950 1850
-F 0 "TP2" V 1904 1908 50  0000 L CNN
-F 1 "5V" V 1995 1908 50  0000 L CNN
-F 2 "TestPoint:TestPoint_2Pads_Pitch2.54mm_Drill0.8mm" H 1950 1850 50  0001 C CNN
-F 3 "~" H 1950 1850 50  0001 C CNN
-	1    1950 1850
-	0    1    1    0
-$EndComp
-Connection ~ 2050 3000
 Wire Wire Line
 	2050 3000 2200 3000
@@
 	1    0    0    -1
 $EndComp
-Wire Wire Line
-	1800 1650 1950 1650
-Connection ~ 1950 1650
 $Comp
 L power:+12V #PWR09
 U 1 1 5C46936E
-P 700 1650
-F 0 "#PWR09" H 700 1500 50  0001 C CNN
-F 1 "+12V" H 715 1823 50  0000 C CNN
-F 2 "" H 700 1650 50  0001 C CNN
-F 3 "" H 700 1650 50  0001 C CNN
-	1    700  1650
-	1    0    0    -1
-$EndComp
-Wire Wire Line
-	850  1650 700  1650
-$Comp
-L power:GND #PWR016
-U 1 1 5C47577B
-P 1950 2150
-F 0 "#PWR016" H 1950 1900 50  0001 C CNN
-F 1 "GND" H 1955 1977 50  0000 C CNN
-F 2 "" H 1950 2150 50  0001 C CNN
-F 3 "" H 1950 2150 50  0001 C CNN
-	1    1950 2150
-	1    0    0    -1
-$EndComp
-Wire Wire Line
-	1950 2150 1950 2050
+P 2400 1650
+F 0 "#PWR09" H 2400 1500 50  0001 C CNN
+F 1 "+12V" H 2415 1823 50  0000 C CNN
+F 2 "" H 2400 1650 50  0001 C CNN
+F 3 "" H 2400 1650 50  0001 C CNN
+	1    2400 1650
+	1    0    0    -1
+$EndComp
 $Comp
 L power:PWR_FLAG #FLG01
@@
 $EndComp
 Connection ~ 3150 1650
-Wire Wire Line
-	1950 1650 2700 1650
 $Comp
 L hackuarium:LOGO #G1
@@
 Wire Wire Line
 	4200 2450 4500 2450
+Wire Wire Line
+	2700 1650 2400 1650
 $EndSCHEMATC
