File: rgb/kicald-old/esp32.sch (KiCad schematic (older format))
At the start: 59 parts, among them J1 5 / 12V, J10 R1, J11 G1, J12 B1, J13 W1, J14 GND1, J15 CONN FT232RL, J16 B2, J17 W2, J18 GND2, J19 R3, J20 G3, J21 B3, J22 W3, J23 GND3, J24 R4, J25 G4, J26 B4, J27 GND4, J3 R2, J4 W1, J5 hole, J6 hole, J7 hole, J8 hole, J9 G2, Q1 BSP75, Q10 BSP75, Q11 BSP75, Q12 BSP75, Q13 BSP75, Q14 BSP75, Q15 BSP75, Q16 BSP75, Q2 BSP75, Q3 BSP75, Q4 BSP75, Q5 BSP75, Q6 BSP75, Q7 BSP75, Q8 BSP75, Q9 BSP75, SW1 RESET, SW2 PROG, U1 ESP32-WROOM-32U, U2 DS18B20, U3 PCA9685PW

Commit message: chore: refactor and finish rgb
Parts:
- removed TP2: 5V, TestPoint:TestPoint_2Pads_Pitch2.54mm_Drill0.8mm, symbol Connector:TestPoint_2Pole
Connections:
- wire segments 134 -> 130
