File: playground/kicad/esp32.sch (KiCad schematic (older format))
At the start: 50 parts, among them J1 5 / 12V, J10 Red, J11 Green, J12 Blue, J13 White, J14 Pad, J15 CONN FT232RL, J16 RJ12-I2C, J17 RJ12-I2C, J2 +12V, J3 Onewire, J4 Onewire, J5 hole, J6 hole, J7 hole, J8 hole, J9 IO_RGBW, Q1 BSP75, Q2 BSP75, Q3 BSP75, Q4 BSP75, SW1 RESET, SW2 PROG, U1 ESP32-WROOM-32U, U2 MS5637, U3 Si7020-A20, U7 DS18B20U, U8 TCS3400

Commit message: fix: close https://github.com/Hackuarium/esp-32wroom/issues/13
Parts:
- Q1, Q2, Q3, Q4: symbol BSP75:BSP75 -> esp32-rescue:BSP75-BSP75
- R4: value 499 -> 1k
Changed lines of the file:
@@
 $EndComp
 $Comp
-L BSP75:BSP75 Q1
+L esp32-rescue:BSP75-BSP75 Q1
 U 1 1 5C3A4B25
 P 7500 4000
@@
 $EndComp
 $Comp
-L BSP75:BSP75 Q2
+L esp32-rescue:BSP75-BSP75 Q2
 U 1 1 5C3A668F
 P 8500 4000
@@
 $EndComp
 $Comp
-L BSP75:BSP75 Q3
+L esp32-rescue:BSP75-BSP75 Q3
 U 1 1 5C3A66DF
 P 9600 4000
@@
 $EndComp
 $Comp
-L BSP75:BSP75 Q4
+L esp32-rescue:BSP75-BSP75 Q4
 U 1 1 5C3A6717
 P 10600 4000
@@
 P 5500 4050
 F 0 "R4" V 5500 4050 50  0000 C CNN
-F 1 "499" V 5600 4050 50  0000 C CNN
+F 1 "1k" V 5600 4050 50  0000 C CNN
 F 2 "Resistor_SMD:R_0805_2012Metric_Pad1.15x1.40mm_HandSolder" V 5430 4050 50  0001 C CNN
 F 3 "~" H 5500 4050 50  0001 C CNN
@@
 Wire Wire Line
 	1750 1650 1950 1650
-$Sheet
-S 5950 1350 800  600
-U 5DE79008
-F0 "ACT4088-33" 50
-F1 "hacki/sheets/ACT4088-33/ACT4088-33.sch" 50
-F2 "VIN" I L 5950 1650 50
-F3 "3.3V" O R 6750 1650 50
-$EndSheet
 Wire Wire Line
 	5500 1650 5950 1650
@@
 Wire Wire Line
 	10150 5150 10150 5300
+$Sheet
+S 5950 1350 800  550
+U 5DEE175C
+F0 "AP7365-33YG" 50
+F1 "hacki/sheets/AP7365-33Y/AP7365-33Y.sch" 50
+F2 "VIN" I L 5950 1650 50
+F3 "VOUT" I R 6750 1650 50
+$EndSheet
 $EndSCHEMATC

Commit message: fix: close https://github.com/Hackuarium/esp-32wroom/issues/8
Changed lines of the file:
@@
 Wire Wire Line
 	4700 1850 5200 1850
-Text GLabel 3950 4150 0    50   Input ~ 0
+Text GLabel 3950 4250 0    50   Input ~ 0
 CHARGING
-Wire Wire Line
-	4000 4150 3950 4150
 $Comp
 L RF_Module:ESP32-WROOM-32U U1
@@
 NoConn ~ 4000 5550
 NoConn ~ 4000 5650
-NoConn ~ 4000 4250
 NoConn ~ 5200 4450
 NoConn ~ 5200 4950
@@
 F3 "VOUT" I R 6750 1650 50
 $EndSheet
+Wire Wire Line
+	3950 4250 4000 4250
+NoConn ~ 4000 4150
 $EndSCHEMATC

Commit message: fix: rename One1 to One3
Changed lines of the file:
@@
 ONE2
 Text Label 5300 4350 0    50   ~ 0
-ONE1
+ONE3
 Text GLabel 5550 5350 2    50   Input ~ 0
 SDA
