File: rgb/kicad/esp32.sch (KiCad schematic (older format))
At the start: 31 parts, among them J1 5 / 12V, J11 +12V, J15 CONN FT232RL, J17 +12V, J2 +12V, J22 +12V, J5 hole, J6 hole, J7 hole, J8 hole, SW1 RESET, SW2 PROG, U1 ESP32-WROOM-32U, U2 MS5637, U3 Si7020-A20, U6 DS18B20, U8 TCS3400

Commit message: fix(rgb): add DTR CSR, pullup IO0
Parts:
- removed D1: D_Schottky, Diode_SMD:D_SOD-123, symbol Device:D_Schottky
- added R1: 10k, Resistor_SMD:R_0805_2012Metric_Pad1.15x1.40mm_HandSolder, symbol Device:R
Connections:
- net labels removed: CHARGING
- no-connect marks 22 -> 31
